File: IGN6.kicad_sch (KiCad schematic)
At the start: 24 parts

Commit message: Rev.D
Parts:
- removed R14 (x6): 0, Resistor_SMD:R_2512_6332Metric, symbol hellen-one-common:Res
- added JP1, JP2, JP3, JP4, JP5, JP6: Jumper_3_Open, Connector_PinHeader_1.27mm:PinHeader_1x03_P1.27mm_Vertical, symbol Jumper:Jumper_3_Open
- Q? (x6): LCSC (none) -> C603080; MyComment DNP -> (none)
Connections:
- net OUT1: now also JP1.3 (B)
- net OUT2: now also JP2.3 (B)
- net OUT3: now also JP3.3 (B)
- net OUT4: now also JP4.3 (B)
- net OUT5: now also JP5.3 (B)
- net OUT6: now also JP6.3 (B)
- net at F9.1: now also JP5.2 (C); no longer R7.2
- net at F10.1: now also JP6.2 (C); no longer R7.2
- net at R7.2: now also JP1.1 (A); no longer F6.1
- net at R7.2: now also JP4.1 (A); no longer F8.1
- net at R7.2: now also JP2.1 (A); no longer F5.1
- net at R7.2: now also JP3.1 (A); no longer F7.1
- new net: F6.1, JP1.2 (C)
- new net: JP6.1 (A), R7.2
- new net: F8.1, JP4.2 (C)
- new net: JP5.1 (A), R7.2
- new net: F5.1, JP2.2 (C)
- new net: F7.1, JP3.2 (C)
Other:
- moved on the sheet: F10, F8, F9, Q?, R7
