File: uaefi.kicad_sch (KiCad schematic)
At the start: 46 parts, among them J1 211PL562L0011, J1 USB_B_Mini, J1 USB_C, J17 Conn_01x06, J3 5569-06A2, J5 Conn_01x05_Male, M1 Module-power_12and5V-0.2, M3 Module-knock-0.2, M3 Module-vr-discrete-0.5, M4 Module-vr-max9924-0.1, M5 Module-wbo-0.5, M6 Module:mega-mcu100/0.3, M7 Module-can-0.1, P1 Pad, P2 Pad, P3 Pad, P4 Pad, P7 Pad, P8 Pad, U4 JDY-33

Commit message: Reev.D update
Parts:
- J3: now left out of the parts list
Changed lines of the file:
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@@
   )
   (symbol (lib_id "Connector_Generic:Conn_02x03_Top_Bottom") (at 92.329 79.756 0) (mirror x) (unit 1)
-    (in_bom yes) (on_board yes) (dnp no)
+    (in_bom no) (on_board yes) (dnp no)
     (property "Reference" "J3" (at 93.599 74.676 0)
       (effects (font (size 1.27 1.27)))

Commit message: Update uaefi.kicad_sch
Parts:
- J3: now in the parts list
Changed lines of the file:
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@@
   )
   (symbol (lib_id "Connector_Generic:Conn_02x03_Top_Bottom") (at 92.329 79.756 0) (mirror x) (unit 1)
-    (in_bom no) (on_board yes) (dnp no)
+    (in_bom yes) (on_board yes) (dnp no)
     (property "Reference" "J3" (at 93.599 74.676 0)
       (effects (font (size 1.27 1.27)))
