File: uaefi.kicad_sch (KiCad schematic)
At the start: 66 parts, among them J1 Conn_02x02_Odd_Even, J1 USB_B_Mini, J1 USB_C, J10 5569-16A2, J11 Conn_02x02_Odd_Even, J12 Conn_02x02_Odd_Even, J13 Conn_02x02_Odd_Even, J14 Conn_02x02_Odd_Even, J15 Conn_02x02_Odd_Even, J16 Conn_02x02_Odd_Even, J17 Conn_01x06, J17 Conn_02x02_Odd_Even, J18 Conn_02x02_Odd_Even, J19 Conn_02x02_Odd_Even, J2 5569-20A2, J20 Conn_02x02_Odd_Even, J21 Conn_02x02_Odd_Even, J22 Conn_02x02_Odd_Even, J24 Conn_02x02_Odd_Even, J3 5569-06A2, J4 5569-08A2, J5 5569-18A2, J5 Conn_01x05_Male, M1 Module-power_12and5V-0.2, M3 Module-knock-0.2, M3 Module-vr-discrete-0.5, M4 Module-vr-max9924-0.1, M5 Module-wbo-0.5, M6 Module:mega-mcu100/0.3, M7 Module-can-0.1, P1 Pad, P2 Pad, P3 Pad, P4 Pad, P7 Pad, P8 Pad, U4 JDY-33

Commit message: Rev.D
Parts:
- removed H3, H4: M3, MountingHole:MountingHole_3.2mm_M3_Pad_Via, symbol Mechanical:MountingHole
- removed J1, J11, J12, J13, J14, J15, J16, J17, J18, J19, J20, J21, J22, J24: Conn_02x02_Odd_Even, Connector_PinSocket_2.54mm:PinSocket_2x02_P2.54mm_Vertical, symbol Connector_Generic:Conn_02x02_Odd_Even
- removed J10: 5569-16A2, Connector_Molex:Molex_Mini-Fit_Jr_5569-16A2_2x08_P4.20mm_Horizontal, symbol Connector_Generic:Conn_02x08_Top_Bottom
- removed J2: 5569-20A2, Connector_Molex:Molex_Mini-Fit_Jr_5569-20A2_2x10_P4.20mm_Horizontal, symbol Connector_Generic:Conn_02x10_Top_Bottom
- removed J4: 5569-08A2, Connector_Molex:Molex_Mini-Fit_Jr_5569-08A2_2x04_P4.20mm_Horizontal, symbol Connector_Generic:Conn_02x04_Top_Bottom
- removed J5: 5569-18A2, Connector_Molex:Molex_Mini-Fit_Jr_5569-18A2_2x09_P4.20mm_Horizontal, symbol Connector_Generic:Conn_02x09_Top_Bottom
- removed R30 (x2): 0, hellen-one-common:R0603, symbol hellen-one-common:Res
- added J1: 211PL562L0011, uaefi-main:211PL562L0011_2, symbol Proteus_Little-eagle-import:211PL562L0011
- added JP1: Jumper_3_Open, Connector_PinHeader_1.27mm:PinHeader_1x03_P1.27mm_Vertical, symbol Jumper:Jumper_3_Open
Connections:
- net +12V: now also J1.P37 (37)
- net +5VP: now also J1.P48 (48), J1.P49 (49)
- net 12V_KEY: now also J1.P36 (36)
- net ADC3: now also JP1.2 (C)
- net CAN+: now also J1.P3 (3)
- net CAN-: now also J1.P2 (2)
- net EGT+: now also J1.P4 (4)
- net EGT-: now also J1.P5 (5)
- net GND: now also J1.P50 (50), J1.P51 (51)
- net GNDA: now also J1.P7 (7), J1.P8 (8)
- net IN_AUX1: now also J1.P56 (56)
- net IN_AUX2: now also J1.P29 (29)
- net IN_AUX3: now also J1.P54 (54)
- net IN_BUTTON1: now also J1.P23 (23)
- net IN_BUTTON2: now also J1.P22 (22)
- net IN_BUTTON3: now also J1.P21 (21)
- net IN_CLT: now also J1.P9 (9)
- net IN_FLEX: now also J1.P13 (13)
- net IN_HALL1: now also J1.P31 (31)
- net IN_HALL2: now also J1.P53 (53)
- net IN_HALL3: now also J1.P52 (52)
- net IN_IAT: now also J1.P10 (10)
- net IN_KNOCK: now also JP1.1 (A)
- net IN_KNOCK_RAW: now also J1.P6 (6)
- net IN_MAP: now also J1.P14 (14)
- net IN_PPS1: now also J1.P11 (11)
- net IN_PPS2: now also J1.P30 (30)
- net IN_TPS1: now also J1.P12 (12)
- net IN_TPS2: now also J1.P55 (55)
- net OUT_DC1+: now also J1.P41 (41)
- net OUT_DC1-: now also J1.P40 (40)
- net OUT_DC2+: now also J1.P38 (38)
- net OUT_DC2-: now also J1.P39 (39)
- net OUT_IGN1: now also J1.P1 (1)
- net OUT_IGN2: now also J1.P28 (28)
- net OUT_IGN3: now also J1.P27 (27)
- net OUT_IGN4: now also J1.P26 (26)
- net OUT_IGN5: now also J1.P25 (25)
- net OUT_IGN6: now also J1.P24 (24)
- net OUT_INJ1: now also J1.P15 (15)
- net OUT_INJ2: now also J1.P16 (16)
- net OUT_INJ3: now also J1.P17 (17)
- net OUT_INJ4: now also J1.P18 (18)
- net OUT_INJ5: now also J1.P19 (19)
- net OUT_INJ6: now also J1.P20 (20)
- net OUT_LS1: now also J1.P46 (46)
- net OUT_LS2: now also J1.P47 (47)
- net OUT_LS3: now also J1.P44 (44)
- net OUT_LS4: now also J1.P45 (45)
- net OUT_LS_HOT1: now also J1.P43 (43)
- net OUT_LS_HOT2: now also J1.P42 (42)
- net VR_DISCRETE+: now also J1.P35 (35)
- net VR_DISCRETE-: now also J1.P34 (34)
- net VR_DISCRETE_A: now also JP1.3 (B)
- net VR_MAX9924+: now also J1.P33 (33)
- net VR_MAX9924-: now also J1.P32 (32)
Other:
- note added: "Move jumper position to use ADC3 for receiving the analog signal VR-DISCRETE instead of the knock signal"
- note added: "Pin Name Recommended function P42 OUT_LS_HOT2 Fan Relay P43 OUT_LS_HOT1 Main Relay P45 OUT_LS4 Fuel Pump Replay P47 OUT_LS2 Idle Air Valve P54 IN_AUX3 Fuel Pressure P22 IN_BUTTON2 A/C Request"
- note removed: "A"
- note removed: "B"
- note removed: "C"
- note removed: "D"
- note removed: "Move the resistor from position R6 to R5 to use ADC3 for receiving the analog signal VR-DISCRETE instead of the knock signal"
- note removed: "Pin 8 may be used for shielding VR signals"
- note removed: "Pin Name Recommended function B8 OUT_LS_HOT2 Fan Relay B9 OUT_LS_HOT1 Main Relay B16 OUT_LS4 Fuel Pump Replay B18 OUT_LS2 Idle Air Valve C8 GND VR Shield C16 IN_AUX3 Fuel Pressure D10 IN_BUTTON2 A/C Request"
- moved on the sheet: BT1, C3, D10, F6, J1, J17, J3, M1, M3, M4, M5, M6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

Commit message: Rev.D update
Parts:
- H1: value M3 -> M4; footprint MountingHole:MountingHole_3.2mm_M3_Pad_Via -> MountingHole:MountingHole_4.3x6.2mm_M4_Pad_Via
- H2: footprint MountingHole:MountingHole_3.2mm_M3_Pad_Via -> MountingHole:MountingHole_4.3x6.2mm_M4_Pad_Via
Other:
- moved on the sheet: H1
Changed lines of the file:
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@@
     )
   )
-  (symbol (lib_id "Mechanical:MountingHole") (at 62.23 394.97 0) (unit 1)
+  (symbol (lib_id "Mechanical:MountingHole") (at 62.23 394.97 180) (unit 1)
     (in_bom yes) (on_board yes) (dnp no) (fields_autoplaced)
-    (property "Reference" "H1" (at 64.77 393.7 0)
-      (effects (font (size 1.27 1.27)) (justify left))
-    )
-    (property "Value" "M3" (at 64.77 396.24 0)
-      (effects (font (size 1.27 1.27)) (justify left))
-    )
-    (property "Footprint" "MountingHole:MountingHole_3.2mm_M3_Pad_Via" (at 62.23 394.97 0)
+    (property "Reference" "H1" (at 64.77 394.335 0)
+      (effects (font (size 1.27 1.27)) (justify right))
+    )
+    (property "Value" "M4" (at 64.77 396.875 0)
+      (effects (font (size 1.27 1.27)) (justify right))
+    )
+    (property "Footprint" "MountingHole:MountingHole_4.3x6.2mm_M4_Pad_Via" (at 62.23 394.97 0)
       (effects (font (size 1.27 1.27)) hide)
     )
@@
       (effects (font (size 1.27 1.27)) (justify left))
     )
-    (property "Footprint" "MountingHole:MountingHole_3.2mm_M3_Pad_Via" (at 62.23 401.32 0)
-      (effects (font (size 1.27 1.27)) hide)
-    )
+    (property "Footprint" "MountingHole:MountingHole_4.3x6.2mm_M4_Pad_Via" (at 62.23 401.32 0)
+      (effects (font (size 1.27 1.27)) hide)
+    )
